File: KiCad/CMS/CMS.kicad_pcb (KiCad board)
At the start: 2 copper layers, 30.5 x 33 mm, 16 parts, among them U1 LTC6090, U2 LTC6090

Commit message: Better schematics + 3D models + New images
Connections:
- net Net-(U1-V+) renamed V+
- net Net-(U1-V-) renamed V-
